File: inchdigits.kicad_pcb (KiCad board)
At the start: 2 copper layers, 99.3 x 56.1 mm, 18 parts, among them J1 Power/Data, J2 Buttons matrix, U1 TM1637

Commit message: Update to KiCad 7, small tweaks
Parts:
- H1, H2, H3, H4: footprint MountingHole:MountingHole_3.5mm -> MountingHole:MountingHole_3.5mm_Pad
- moved REF** 1.27 mm to (111.8, 94.0)
