File: inchdigits.kicad_sch (KiCad schematic)
At the start: 17 parts, among them J1 Power/Data, J2 Buttons matrix, U1 TM1637

Commit message: Update to KiCad 7, small tweaks
Parts:
- H1, H2, H3, H4: footprint MountingHole:MountingHole_3.5mm -> MountingHole:MountingHole_3.5mm_Pad
